File: PCB_prototype1/PCB_prototype1.kicad_sch (KiCad schematic)
At the start: 6 parts, among them U1 LSM6DSV16X

Commit message: Schematic updated
Parts:
- added C4, C5: 10uF, symbol Device:C_Small
- added C6: 1uF, symbol Device:C_Small
- added C7, C8: 4.7uF, symbol Device:C_Small
- added J2: Conn_01x11_Pin, symbol Connector:Conn_01x11_Pin
- added U2: VL53L9CX, symbol Lidar:VL53L9CX_large
- R1, R2: value 10k -> 2.2k
Connections:
- net +3.3V: now also J2.1 (Pin_1)
- net GND: now also C4.2, C5.2, C6.2, C7.2, C8.2, J2.11 (Pin_11), U2.A1 (VSS), U2.A2 (VSS_DRIVER), U2.A3 (VSS_DRIVER), U2.A4 (VSS), U2.A7 (VSS), U2.B4 (VSS), U2.B5 (VSS), U2.B6 (VSS), U2.B7 (VSS), U2.B8 (VSS), U2.B9 (VSS), U2.C1 (VSS), U2.D4 (VSS), U2.D5 (VSS), U2.D6 (VSS), U2.D7 (VSS), U2.D8 (VSS), U2.D9 (VSS), U2.E1 (VSS), U2.E10 (VSS), U2.E2 (VSS), U2.E4 (VSS), U2.E5 (VSS), U2.E9 (VSS)
- net GPIO_EXTI: now also J2.10 (Pin_10)
- net i2c_SCL: now also J2.9 (Pin_9)
- net i2c_SDA: now also J2.8 (Pin_8)
- new net +3V3: C4.1, C5.1, C6.1, C7.1, U2.B1 (VBAT_LDD), U2.D1 (VBAT_RX), U2.E6 (AVDD), U2.E7 (AVDD), U2.E8 (IOVDD)
- new net AP_CLK: J2.4 (Pin_4), U2.E11 (AP_CLK)
- new net CLK_N: U2.A9 (CLK_N)
- new net CLK_P: U2.A8 (CLK_P)
- new net DATA_N: U2.A6 (DATA_N)
- new net DATA_P: U2.A5 (DATA_P)
- new net DVDD: C8.1, U2.C12 (DVDD)
- new net INTR: J2.7 (Pin_7), U2.A10 (INTR)
- new net SYNC_IN: J2.6 (Pin_6), U2.D12 (SYNC_IN)
- new net XSHUT: J2.5 (Pin_5), U2.B12 (XSHUT)
- new net i3c_SCL: J2.2 (Pin_2), U2.A11 (SCL)
- new net i3c_SDA: J2.3 (Pin_3), U2.A12 (SDA)

Commit message: ajout de rapport de seance
Parts:
- added IC1: VL53L9CX, VL53L9CX, symbol VL53L9CX:VL53L9CX

Commit message: update
Connections:
- net +3V3: now also IC1.D1 (VBAT_RX)
- net DVDD: now also IC1.C12 (DVDD)
- net GND: now also IC1.A1 (VSS_1), IC1.A2 (VSS_DRIVER_1), IC1.A3 (VSS_DRIVER_2), IC1.A4 (VSS_2), IC1.B4 (VSS_4), IC1.B5 (VSS_5), IC1.B6 (VSS_6), IC1.B7 (VSS_7), IC1.B8 (VSS_8), IC1.B9 (VSS_9), IC1.C1 (VSS_10), IC1.D4 (VSS_11), IC1.D5 (VSS_12), IC1.D6 (VSS_13), IC1.D7 (VSS_14), IC1.D8 (VSS_15), IC1.D9 (VSS_16), IC1.E1 (VSS_17), IC1.E10 (VSS_22), IC1.E2 (VSS_18), IC1.E9 (VSS_21)
- net SYNC_IN: now also IC1.D12 (SYNC_IN)
- no-connect marks 5 -> 6

Commit message: .
Parts:
- removed IC1: VL53L9CX, VL53L9CX, symbol VL53L9CX:VL53L9CX
- added IC1: ST67W611M1A6B, ST67W611M1A6B, symbol carte_wifi:ST67W611M1A6B
Connections:
- net +3V3: no longer C6.1, U2.E8 (IOVDD)
- new net +1V8: C6.1, U2.E8 (IOVDD)
- no-connect marks 6 -> 5
Other:
- moved on the sheet: J2
